File: EAGLE/ENGI301_Maze_Project_v2.sch (EAGLE design)
At the start: 27 parts, among them U1 MOD-LED8X8RGB-CONN, U2 MOD-LED8X8RGB-CONN, U3 POCKETBEAGLE

Commit message: Added pictures of top and bottom layer.
Other:
- note added: "Only two LED arrays are connected to board directly; Other two are daisy-chained"
Changed lines of the file:
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@@
 <drawing>
 <settings>
-<setting alwaysvectorfont="yes"/>
+<setting alwaysvectorfont="no"/>
 <setting verticaltext="up"/>
 </settings>
@@
 Button</text>
 <text x="114.3" y="190.5" size="5.08" layer="95">Buzzer</text>
+<text x="314.96" y="162.56" size="1.778" layer="91">Only two LED arrays are connected to
+board directly;
+Other two are daisy-chained</text>
 </plain>
 <instances>
